File: Arduino_Flight_Controller v1.1/Arduino_Flight_Controller.kicad_pcb (KiCad board)
At the start: 2 copper layers, 55.5 x 50.4 mm, 17 parts, among them J1 MPU_9250, J2 RC_BAT, J3 RF_PPM, J4 BMP_280, J5 ESC_Signal, J6 HC-SRO4, J7 Screw_Terminal_01x02, U1 AMS1117-5.0

Commit message: first commit
Other:
- net class Default removed
